Commit message: Inicio robot 2 ruedas

File: src/mlp2wr_description/urdf/macros.xacro (robot description, xacro)
@@ -12,5 +12,5 @@
 		      <origin rpy="0 1.5707 1.5707" xyz="0 0 0"/>
 		      <geometry>
-			<cylinder length="0.025" radius="0.035"/>
+			<cylinder length="0.04" radius="0.1"/>
 		      </geometry>
 		    </collision>
@@ -18,15 +18,14 @@
 		      <origin rpy="0 1.5707 1.5707" xyz="0 0 0"/>
 		      <geometry>
-							<cylinder length="0.025" radius="0.035"/>
+			<cylinder length="0.04" radius="0.1"/>
 		      </geometry>
 		    </visual>
   		</link>
 	</macro>
-<!--Macro para los joints-->
 <macro name = "joint_wheel" params = "name child origin_xyz">
  <joint name="${name}" type="continuous">
     <origin rpy="0 0 0" xyz="${origin_xyz}"/>
     <child link="${child}"/>
-    <parent link="base_link"/>
+    <parent link="link_chassis"/>
     <axis rpy="0 0 0" xyz="0 1 0"/>
     <limit effort="10000" velocity="1000"/>

File: src/mlp2wr_description/urdf/mlp2wr.xacro (robot description, xacro)
@@ -5,6 +5,7 @@
   <xacro:include filename="$(find mlp2wr_description)/urdf/macros.xacro"/>
 <!--Cuerpo para el chasis -->
-  <link name="base_link">
-    <!-- Inercial-->
+  <link name="link_chassis">
+    <!-- pose and inertial -->
+    <pose>0 0 1 0 0 0</pose>
     <inertial>
       <mass value="5"/>
@@ -12,32 +13,52 @@
       <inertia ixx="0.0395416666667" ixy="0" ixz="0" iyy="0.106208333333" iyz="0" izz="0.106208333333"/>
     </inertial>
-    <!-- Colision -->
-    <collision name="collision_base">
+    <!-- body -->
+    <collision name="collision_chassis">
       <geometry>
-        <box size="0.1 0.15 0.02"/>
+        <box size="0.5 0.3 0.07"/>
       </geometry>
     </collision>
-    <!--Visual-->
     <visual>
       <origin rpy="0 0 0" xyz="0 0 0"/>
       <geometry>
-        <box size="0.1 0.15 0.02"/>
+        <box size="0.5 0.3 0.07"/>
       </geometry>
       <material name="blue"/>
     </visual>
-</link>
+    <!-- caster front -->
+    <collision name="caster_front_collision">
+      <origin rpy=" 0 0 0" xyz="0.35 0 -0.05"/>
+      <geometry>
+        <sphere radius="0.05"/>
+      </geometry>
+      <surface>
+        <friction>
+          <ode>
+            <mu>0</mu>
+            <mu2>0</mu2>
+            <slip1>1.0</slip1>
+            <slip2>1.0</slip2>
+          </ode>
+        </friction>
+      </surface>
+    </collision>
+    <visual name="caster_front_visual">
+      <origin rpy=" 0 0 0" xyz="0.2 0 -0.05"/>
+      <geometry>
+        <sphere radius="0.05"/>
+      </geometry>
+    </visual>
+  </link>
 <!--Cuerpo para el sensor-->
 <link name="sensor_laser">
-  <!--Inercial-->
     <inertial>
         <origin xyz="0 0 0" rpy="0 0 0" />
         <mass value="1" />
-        <xacro:cylinder_inertia mass="1" r="0.014" l="0.012" />
+        <xacro:cylinder_inertia mass="1" r="0.05" l="0.1" />
     </inertial>
-<!--Visual-->
     <visual>
         <origin xyz="0 0 0" rpy="0 0 0" />
         <geometry>
-        <cylinder radius="0.014" length="0.012"/>
+        <cylinder radius="0.05" length="0.1"/>
         </geometry>
         <material name="white" />
@@ -46,27 +67,17 @@
         <origin xyz="0 0 0" rpy="0 0 0"/>
         <geometry>
-        <cylinder  radius="0.014" length="0.012"/>
+        <cylinder radius="0.05" length="0.1"/>
         </geometry>
     </collision>
-</link>
+    </link>
 <!--Joint para el sensor -->
 <joint name = "joint_sensor_laser" type = "fixed">
-	<origin xyz = "0 0.106 0.032" rpy = "0 0 0 "/>
-	<parent link = "base_link"/>
+	<origin xyz = "0.15 0 0.05" rpy = "0 0 0 "/>
+	<parent link = "link_chassis"/>
 	<child link = "sensor_laser"/>
 </joint>
-              <!--Crear las ruedas-->
-<!--Ruedas delanteras-->
-<xacro:link_wheel name ="link_wheelFL"/>
-<xacro:link_wheel name ="link_wheelFR"/>
-<!--Ruedas traseras-->
-<xacro:link_wheel name ="link_wheelBL"/>
-<xacro:link_wheel name ="link_wheelBR"/>
-<!-- CRear las uniones entre el chasis y las ruedas-->
-<!--Uniones  delanteras-->
- <xacro:joint_wheel name ="joint_wheelFL" child = "link_wheelFL" origin_xyz = "-0.05 0.075 0"/>
- <xacro:joint_wheel name = "joint_wheelFR" child = "link_wheelFR" origin_xyz = "0.05 0.075 0"/>
-<!--Uniones  delanteras-->
- <xacro:joint_wheel name ="joint_wheelBL" child = "link_wheelBL" origin_xyz = "-0.05 -0.075 0"/>
- <xacro:joint_wheel name = "joint_wheelBR" child = "link_wheelBR" origin_xyz = "0.05 -0.075 0"/>
+ <xacro:link_wheel name ="link_right_wheel"/>
+ <xacro:joint_wheel name ="joint_right_wheel" child = "link_right_wheel" origin_xyz = "-0.05 0.2 0"/>
+ <xacro:link_wheel name ="link_left_wheel"/>
+ <xacro:joint_wheel name = "joint_left_wheel" child = "link_left_wheel" origin_xyz = "-0.05 -0.2 0"/>
 </robot>
